File: 555-bipolar/555bip.kicad_sch (KiCad schematic)
At the start: 50 parts, among them Q1 PN, Q10 NP, Q11 PN, Q12 NP, Q13 NP, Q14 NP, Q15 PN, Q16 PN, Q17 PN, Q18 NP, Q19 NP, Q2 NP, Q20 PN, Q21 NP, Q22 NP, Q23 PN, Q24 NP, Q25 PN, Q26 NP, Q27 NP, Q28 NP, Q29 NP, Q3 PN, Q30 PN, Q31 NP, Q32 NP, Q4 NP, Q5 PN, Q6 NP, Q7 PN, Q8 PN, Q9 PN

Commit message: Updated to KiCad 8, changed simulation duration for better plot
Parts:
- Q1, Q11, Q15, Q16, Q17, Q20, Q23, Q25, Q3, Q30, Q5, Q7, Q8, Q9: Spice_Lib_File bipmod.lib -> (none); Spice_Model PN -> (none); Spice_Netlist_Enabled Y -> (none); Spice_Primitive Q -> (none)
- Q10, Q12, Q13, Q14, Q18, Q19, Q2, Q21, Q22, Q24, Q26, Q27, Q28, Q29, Q31, Q32, Q4, Q6: Spice_Lib_File bipmod.lib -> (none); Spice_Model NP -> (none); Spice_Netlist_Enabled Y -> (none); Spice_Primitive Q -> (none)
- V1: Spice_Model 15 -> (none); Spice_Netlist_Enabled Y -> (none); Spice_Primitive V -> (none)
- V3: Spice_Model pulse(0 15 0 1u 1u 5m 10m) -> (none); Spice_Netlist_Enabled Y -> (none); Spice_Primitive V -> (none)
Other:
- note added: ".tran 1u 12m"
- note removed: ".tran 1u 30m"
